File: EAGLE Board Designs/Main ECU/MainECU rev9.sch (EAGLE design)
At the start: 203 parts, among them J1 JUMPER, J2 JUMPER, J3 JUMPER, J4 JUMPER, J5 JUMPER, J6 JUMPER, J7 JUMPER, J8 JUMPER, P1 SOLDER_PAD, P2 SOLDER_PAD, Q12 P-CHANNEL_MOSFET_DMP3099L-7, X1 CONNECTOR-37, X2 CONNECTOR-4AUTOSPORT, X3 CONNECTOR-4NANO-FIT-VERTICAL-4, X4 CONNECTOR-4NANO-FIT-VERTICAL-4

Commit message: Update MainECU rev9.sch
Parts:
- added R13: 20, HyTechDevices:RESISTOR0805-RES
Connections:
- new net N$12: R13.1, U$14.4
- net GND: now also R13.2; no longer U$14.4
Changed lines of the file:
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@@
 <part name="R12" library="HyTechDevices" deviceset="RESISTOR" device="0805-RES" value="2k"/>
 <part name="GND11" library="HyTechSymbols" deviceset="GND" device=""/>
+<part name="R13" library="HyTechDevices" deviceset="RESISTOR" device="0805-RES" value="20"/>
 </parts>
 <sheets>
@@
 <attribute name="VALUE" x="76.2" y="177.8" size="1.778" layer="96"/>
 </instance>
-<instance part="GND19" gate="1" x="119.38" y="195.58" smashed="yes">
-<attribute name="VALUE" x="116.84" y="193.04" size="1.778" layer="96"/>
+<instance part="GND19" gate="1" x="134.62" y="203.2" smashed="yes" rot="R180">
+<attribute name="VALUE" x="137.16" y="205.74" size="1.778" layer="96" rot="R180"/>
 </instance>
 <instance part="R17" gate="G$1" x="137.16" y="180.34" smashed="yes">
@@
 <attribute name="VALUE" x="96.52" y="238.76" size="1.778" layer="96" rot="R270"/>
 </instance>
+<instance part="R13" gate="G$1" x="124.46" y="198.12" smashed="yes">
+<attribute name="NAME" x="120.65" y="199.6186" size="1.778" layer="95"/>
+<attribute name="VALUE" x="120.65" y="194.818" size="1.778" layer="96"/>
+</instance>
 </instances>
 <busses>
@@
 </segment>
 <segment>
-<pinref part="GND19" gate="1" pin="GND"/>
-<wire x1="119.38" y1="198.12" x2="114.3" y2="198.12" width="0.1524" layer="91"/>
-<pinref part="U$14" gate="G$1" pin="4"/>
-</segment>
-<segment>
 <pinref part="R58" gate="G$1" pin="2"/>
 <wire x1="271.78" y1="68.58" x2="271.78" y2="66.04" width="0.1524" layer="91"/>
@@
 <wire x1="104.14" y1="236.22" x2="101.6" y2="236.22" width="0.1524" layer="91"/>
 </segment>
+<segment>
+<pinref part="R13" gate="G$1" pin="2"/>
+<pinref part="GND19" gate="1" pin="GND"/>
+<wire x1="129.54" y1="198.12" x2="134.62" y2="198.12" width="0.1524" layer="91"/>
+<wire x1="134.62" y1="198.12" x2="134.62" y2="200.66" width="0.1524" layer="91"/>
+</segment>
 </net>
 <net name="+12V" class="0">
@@
 </segment>
 </net>
+<net name="N$12" class="0">
+<segment>
+<pinref part="U$14" gate="G$1" pin="4"/>
+<pinref part="R13" gate="G$1" pin="1"/>
+<wire x1="114.3" y1="198.12" x2="119.38" y2="198.12" width="0.1524" layer="91"/>
+</segment>
+</net>
