File: EAGLE Board Designs/Dashboard/Dashboard rev2.brd (EAGLE design)
At the start: 177.4 x 27.1 mm, 54 parts, among them J1 AVR-ISP-HEADER, X1 CONNECTOR-6NANO-FIT_VERTICAL-6

Commit message: Added 4 pin conector
Parts:
- added X2: CONNECTOR-4NANO-FIT-VERTICAL-4, HyTechDevices:NANO-FIT_VERTICAL-4
Connections:
- new net WHEEL_POSITION_READ\: X2.P$3
- net +5V: now also X2.P$1
- net GND: now also X2.P$2
