File: EAGLE Board Designs/Dashboard/Dashboard rev2.sch (EAGLE design)
At the start: 54 parts, among them J1 AVR-ISP-HEADER, X1 CONNECTOR-6NANO-FIT_VERTICAL-6

Commit message: Added 4 pin conector
Parts:
- added X2: CONNECTOR-4NANO-FIT-VERTICAL-4, HyTechDevices:CONNECTOR-4NANO-FIT-VERTICAL-4
Connections:
- new net WHEEL_POSITION_READ\: X2-3.S
- net +5V: now also X2-1.S
- net GND: now also X2-2.S
Other:
- moved on the sheet: C1, C7, LM340
Changed lines of the file:
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@@
 <part name="GND17" library="HyTechSymbols" deviceset="GND" device=""/>
 <part name="LM340" library="HyTechDevices" deviceset="LM340" device=""/>
+<part name="X2" library="HyTechDevices" deviceset="CONNECTOR-4" device="NANO-FIT-VERTICAL-4"/>
+<part name="P+12" library="supply1" library_urn="urn:adsk.eagle:library:371" deviceset="+5V" device=""/>
+<part name="GND18" library="HyTechSymbols" deviceset="GND" device=""/>
 </parts>
 <sheets>
@@
 <attribute name="VALUE" x="193.04" y="152.4" size="1.778" layer="96" rot="R180"/>
 </instance>
-<instance part="P+6" gate="1" x="35.56" y="167.64" smashed="yes">
-<attribute name="VALUE" x="33.02" y="170.18" size="1.778" layer="96"/>
-</instance>
-<instance part="P+7" gate="1" x="55.88" y="167.64" smashed="yes">
-<attribute name="VALUE" x="58.42" y="170.18" size="1.778" layer="96" rot="R180"/>
-</instance>
-<instance part="GND7" gate="1" x="45.72" y="144.78" smashed="yes">
-<attribute name="VALUE" x="43.18" y="142.24" size="1.778" layer="96"/>
-</instance>
-<instance part="C1" gate="G$1" x="35.56" y="157.48" smashed="yes" rot="R180">
-<attribute name="NAME" x="34.036" y="154.559" size="1.778" layer="95" rot="R180"/>
-<attribute name="VALUE" x="34.036" y="159.639" size="1.778" layer="96" rot="R180"/>
-</instance>
-<instance part="C7" gate="G$1" x="55.88" y="154.94" smashed="yes">
-<attribute name="NAME" x="57.404" y="157.861" size="1.778" layer="95"/>
-<attribute name="VALUE" x="57.404" y="152.781" size="1.778" layer="96"/>
+<instance part="P+6" gate="1" x="53.34" y="160.02" smashed="yes">
+<attribute name="VALUE" x="50.8" y="162.56" size="1.778" layer="96"/>
+</instance>
+<instance part="P+7" gate="1" x="73.66" y="160.02" smashed="yes">
+<attribute name="VALUE" x="76.2" y="162.56" size="1.778" layer="96" rot="R180"/>
+</instance>
+<instance part="GND7" gate="1" x="63.5" y="137.16" smashed="yes">
+<attribute name="VALUE" x="60.96" y="134.62" size="1.778" layer="96"/>
+</instance>
+<instance part="C1" gate="G$1" x="53.34" y="149.86" smashed="yes" rot="R180">
+<attribute name="NAME" x="51.816" y="146.939" size="1.778" layer="95" rot="R180"/>
+<attribute name="VALUE" x="51.816" y="152.019" size="1.778" layer="96" rot="R180"/>
+</instance>
+<instance part="C7" gate="G$1" x="73.66" y="147.32" smashed="yes">
+<attribute name="NAME" x="75.184" y="150.241" size="1.778" layer="95"/>
+<attribute name="VALUE" x="75.184" y="145.161" size="1.778" layer="96"/>
 </instance>
 <instance part="X1" gate="-1" x="48.26" y="200.66" smashed="yes" rot="MR0">
@@
 <attribute name="VALUE" x="157.48" y="35.56" size="1.778" layer="96"/>
 </instance>
-<instance part="LM340" gate="G$1" x="45.72" y="162.56" smashed="yes">
-<attribute name="NAME" x="48.26" y="154.94" size="1.778" layer="95"/>
-<attribute name="VALUE" x="48.26" y="152.4" size="1.778" layer="96"/>
+<instance part="LM340" gate="G$1" x="63.5" y="154.94" smashed="yes">
+<attribute name="NAME" x="66.04" y="147.32" size="1.778" layer="95"/>
+<attribute name="VALUE" x="66.04" y="144.78" size="1.778" layer="96"/>
+</instance>
+<instance part="X2" gate="-1" x="43.18" y="175.26" smashed="yes" rot="R180">
+<attribute name="NAME" x="40.64" y="176.022" size="1.524" layer="95" rot="R180"/>
+<attribute name="VALUE" x="46.482" y="178.943" size="1.778" layer="96" rot="R180"/>
+</instance>
+<instance part="X2" gate="-2" x="43.18" y="172.72" smashed="yes" rot="R180">
+<attribute name="NAME" x="40.64" y="173.482" size="1.524" layer="95" rot="R180"/>
+</instance>
+<instance part="X2" gate="-3" x="43.18" y="170.18" smashed="yes" rot="R180">
+<attribute name="NAME" x="40.64" y="170.942" size="1.524" layer="95" rot="R180"/>
+</instance>
+<instance part="X2" gate="-4" x="43.18" y="167.64" smashed="yes" rot="R180">
+<attribute name="NAME" x="40.64" y="168.402" size="1.524" layer="95" rot="R180"/>
+</instance>
+<instance part="P+12" gate="1" x="50.8" y="180.34" smashed="yes">
+<attribute name="VALUE" x="50.8" y="182.88" size="1.778" layer="96" rot="R180"/>
+</instance>
+<instance part="GND18" gate="1" x="60.96" y="175.26" smashed="yes">
+<attribute name="VALUE" x="58.42" y="172.72" size="1.778" layer="96"/>
 </instance>
 </instances>
@@
 </segment>
 <segment>
-<wire x1="45.72" y1="154.94" x2="45.72" y2="149.86" width="0.1524" layer="91"/>
-<wire x1="45.72" y1="149.86" x2="45.72" y2="147.32" width="0.1524" layer="91"/>
-<wire x1="43.18" y1="154.94" x2="43.18" y2="149.86" width="0.1524" layer="91"/>
-<wire x1="43.18" y1="149.86" x2="45.72" y2="149.86" width="0.1524" layer="91"/>
-<junction x="45.72" y="149.86"/>
+<wire x1="63.5" y1="147.32" x2="63.5" y2="142.24" width="0.1524" layer="91"/>
+<wire x1="63.5" y1="142.24" x2="63.5" y2="139.7" width="0.1524" layer="91"/>
+<wire x1="60.96" y1="147.32" x2="60.96" y2="142.24" width="0.1524" layer="91"/>
+<wire x1="60.96" y1="142.24" x2="63.5" y2="142.24" width="0.1524" layer="91"/>
+<junction x="63.5" y="142.24"/>
 <pinref part="GND7" gate="1" pin="GND"/>
 <pinref part="C1" gate="G$1" pin="1"/>
-<wire x1="35.56" y1="152.4" x2="35.56" y2="149.86" width="0.1524" layer="91"/>
-<wire x1="35.56" y1="149.86" x2="43.18" y2="149.86" width="0.1524" layer="91"/>
-<junction x="43.18" y="149.86"/>
+<wire x1="53.34" y1="144.78" x2="53.34" y2="142.24" width="0.1524" layer="91"/>
+<wire x1="53.34" y1="142.24" x2="60.96" y2="142.24" width="0.1524" layer="91"/>
+<junction x="60.96" y="142.24"/>
 <pinref part="C7" gate="G$1" pin="2"/>
-<wire x1="55.88" y1="152.4" x2="55.88" y2="149.86" width="0.1524" layer="91"/>
-<wire x1="55.88" y1="149.86" x2="45.72" y2="149.86" width="0.1524" layer="91"/>
+<wire x1="73.66" y1="144.78" x2="73.66" y2="142.24" width="0.1524" layer="91"/>
+<wire x1="73.66" y1="142.24" x2="63.5" y2="142.24" width="0.1524" layer="91"/>
 <pinref part="LM340" gate="G$1" pin="GND"/>
 <pinref part="LM340" gate="G$1" pin="GND1"/>
@@
 <wire x1="160.02" y1="40.64" x2="157.48" y2="40.64" width="0.1524" layer="91"/>
 </segment>
+<segment>
+<pinref part="X2" gate="-2" pin="S"/>
+<wire x1="45.72" y1="172.72" x2="53.34" y2="172.72" width="0.1524" layer="91"/>
+<wire x1="53.34" y1="172.72" x2="53.34" y2="177.8" width="0.1524" layer="91"/>
+<pinref part="GND18" gate="1" pin="GND"/>
+<wire x1="53.34" y1="177.8" x2="60.96" y2="177.8" width="0.1524" layer="91"/>
+</segment>
 </net>
 <net name="+5V" class="0">
@@
 </segment>
 <segment>
-<wire x1="53.34" y1="162.56" x2="55.88" y2="162.56" width="0.1524" layer="91"/>
+<wire x1="71.12" y1="154.94" x2="73.66" y2="154.94" width="0.1524" layer="91"/>
 <pinref part="P+7" gate="1" pin="+5V"/>
-<wire x1="55.88" y1="162.56" x2="55.88" y2="165.1" width="0.1524" layer="91"/>
+<wire x1="73.66" y1="154.94" x2="73.66" y2="157.48" width="0.1524" layer="91"/>
 <pinref part="C7" gate="G$1" pin="1"/>
-<wire x1="55.88" y1="162.56" x2="55.88" y2="160.02" width="0.1524" layer="91"/>
-<junction x="55.88" y="162.56"/>
+<wire x1="73.66" y1="154.94" x2="73.66" y2="152.4" width="0.1524" layer="91"/>
+<junction x="73.66" y="154.94"/>
 <pinref part="LM340" gate="G$1" pin="OUT"/>
 </segment>
@@
 <wire x1="241.3" y1="66.04" x2="238.76" y2="66.04" width="0.1524" layer="91"/>
 </segment>
+<segment>
+<pinref part="P+12" gate="1" pin="+5V"/>
+<pinref part="X2" gate="-1" pin="S"/>
+<wire x1="50.8" y1="177.8" x2="50.8" y2="175.26" width="0.1524" layer="91"/>
+<wire x1="50.8" y1="175.26" x2="45.72" y2="175.26" width="0.1524" layer="91"/>
+</segment>
 </net>
 <net name="SCK" class="0">
@@
 <net name="+12V" class="0">
 <segment>
-<wire x1="38.1" y1="162.56" x2="35.56" y2="162.56" width="0.1524" layer="91"/>
+<wire x1="55.88" y1="154.94" x2="53.34" y2="154.94" width="0.1524" layer="91"/>
 <pinref part="P+6" gate="1" pin="+12V"/>
-<wire x1="35.56" y1="162.56" x2="35.56" y2="165.1" width="0.1524" layer="91"/>
+<wire x1="53.34" y1="154.94" x2="53.34" y2="157.48" width="0.1524" layer="91"/>
 <pinref part="C1" gate="G$1" pin="2"/>
-<wire x1="35.56" y1="160.02" x2="35.56" y2="162.56" width="0.1524" layer="91"/>
-<junction x="35.56" y="162.56"/>
+<wire x1="53.34" y1="152.4" x2="53.34" y2="154.94" width="0.1524" layer="91"/>
+<junction x="53.34" y="154.94"/>
 <pinref part="LM340" gate="G$1" pin="IN"/>
 </segment>
@@
 </segment>
 </net>
+<net name="WHEEL_POSITION_READ\" class="0">
+<segment>
+<pinref part="X2" gate="-3" pin="S"/>
+<wire x1="45.72" y1="170.18" x2="48.26" y2="170.18" width="0.1524" layer="91"/>
+<label x="48.26" y="170.18" size="1.27" layer="95" xref="yes"/>
+</segment>
+</net>
